File: kicad/motherboard/CPU_logic.sch (KiCad schematic (older format))
At the start: 6 parts, among them U27 SN74ALVC00, U28 SN74ALVC00, U29 SN74ALVC00, U30 SN74ALVC00, U31 SN74ALVC00, U32 SN74ALVC00

Commit message: Readme updates (#6)
* Readme intro section

* Board revisions for manufacturing, add digikey PNs to all, added logo.
Parts:
- U27, U28, U29, U30, U31, U32: Digikey PN (none) -> 296-5104-1-ND
Changed lines of the file:
@@
 F 2 "Package_SO:TSSOP-14_4.4x5mm_P0.65mm" H 6500 2550 50  0001 C CNN
 F 3 "" H 6750 4050 50  0001 C CNN
+F 4 "296-5104-1-ND" H 0   0   50  0001 C CNN "Digikey PN"
 	1    6750 4050
 	1    0    0    -1
@@
 F 2 "Package_SO:TSSOP-14_4.4x5mm_P0.65mm" H 2200 1900 50  0001 C CNN
 F 3 "" H 2450 3400 50  0001 C CNN
+F 4 "296-5104-1-ND" H 0   0   50  0001 C CNN "Digikey PN"
 	1    2450 3400
 	1    0    0    -1
@@
 F 2 "Package_SO:TSSOP-14_4.4x5mm_P0.65mm" H 2050 -250 50  0001 C CNN
 F 3 "" H 2300 1250 50  0001 C CNN
+F 4 "296-5104-1-ND" H 0   0   50  0001 C CNN "Digikey PN"
 	1    2300 1250
 	1    0    0    -1
@@
 F 2 "Package_SO:TSSOP-14_4.4x5mm_P0.65mm" H 4450 -250 50  0001 C CNN
 F 3 "" H 4700 1250 50  0001 C CNN
+F 4 "296-5104-1-ND" H 0   0   50  0001 C CNN "Digikey PN"
 	1    4700 1250
 	1    0    0    -1
@@
 F 2 "Package_SO:TSSOP-14_4.4x5mm_P0.65mm" H 6800 -250 50  0001 C CNN
 F 3 "" H 7050 1250 50  0001 C CNN
+F 4 "296-5104-1-ND" H 0   0   50  0001 C CNN "Digikey PN"
 	1    7050 1250
 	1    0    0    -1
@@
 F 2 "Package_SO:TSSOP-14_4.4x5mm_P0.65mm" H 9200 -250 50  0001 C CNN
 F 3 "" H 9450 1250 50  0001 C CNN
+F 4 "296-5104-1-ND" H 0   0   50  0001 C CNN "Digikey PN"
 	1    9450 1250
 	1    0    0    -1
