File: kicad/motherboard/motherboard.kicad_pcb (KiCad board)
At the start: 4 copper layers, 53 parts, among them J1 DB37_Female, J10 DB37_Female, J11 DB37_Female, J12 Barrel_Jack, J13 TSR 1-2433, J2 DB37_Female, J3 DB37_Female, J4 DB37_Female, J5 DB37_Female, J6 DB25_Female, J7 DB37_Female, J8 DB25_Female, J9 DB9_Female, SW1 SW_SPST, U1 SN74ALVC00, U10 SN74ALVC00, U11 SN74ALVC00, U12 SN74ALVC00, U13 SN74ALVC00, U14 SN74ALVC00, U15 SN74ALVC00, U16 SN74ALVC00, U17 SN74ALVC00, U18 SN74ALVC00, U19 SN74ALVC00, U2 SN74ALVC00, U20 SN74ALVC00, U21 SN74ALVC00, U22 SN74ALVC00, U23 SN74ALVC00, U24 SN74ALVC00, U25 SN74ALVC00, U26 SN74ALVC00, U27 SN74ALVC00, U28 SN74ALVC00, U29 SN74ALVC00, U3 SN74ALVC00, U30 SN74ALVC00, U31 SN74ALVC00, U32 SN74ALVC00, U4 SN74ALVC00, U5 SN74ALVC00, U6 SN74ALVC00, U7 SN74ALVC00, U8 SN74ALVC00, U9 SN74ALVC00

Commit message: Motherboard fully routed, PCB layout done
Parts:
- moved U30 277.9 mm to (391.8, 276.9)
- moved U32 276.5 mm to (455.9, 209.6)
- moved U29 267.7 mm to (382.9, 276.9)
- moved U28 264.8 mm to (374.0, 276.9)
- moved U27 255.0 mm to (365.1, 276.9)
- moved U31 149.4 mm to (344.2, 151.1)
- moved U14 43.2 mm to (455.9, 198.8)
- moved U15 40.6 mm to (455.9, 191.8)
- moved U16 35.6 mm to (455.9, 184.8)
- moved U17 33.1 mm to (455.9, 177.8)
- moved U18 28.0 mm to (455.9, 170.8)
- moved U19 25.7 mm to (455.9, 163.8)
- moved U20 20.4 mm to (455.9, 156.8)
- moved U21 18.5 mm to (455.9, 149.9)
- moved SW1 13.4 mm to (450.0, 255.8)
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Connections:
- J8 pad 17: clk_b -> clk_a
- J8 pad 5: clk_a -> clk_b
- R2 pad 1: reset -> +3V3
- R2 pad 2: GND -> reset
- SW1 pad 1: reset -> GND
- SW1 pad 2: +3V3 -> reset
Routing:
- net clk_a: track 0.00 -> 792.7 mm, vias 0 -> 4
- net inst_15: track 286.6 -> 684.6 mm, vias 0 -> 20
- net clk_b: track 0.00 -> 395.7 mm, vias 0 -> 3
- net inst_12: track 286.6 -> 661.6 mm, vias 0 -> 19
- net reset: track 0.00 -> 361.5 mm, vias 0 -> 3
- net pc_inc: track 0.00 -> 345.6 mm, vias 0 -> 3
- net alu_zero: track 0.00 -> 178.7 mm, vias 0 -> 5
- net /Mux_16bit/not_sel: track 0.00 -> 176.8 mm, vias 0 -> 14
- net /sheet5EAF90EF/not_sel: track 0.00 -> 172.1 mm, vias 0 -> 12
- net inst_4: track 286.6 -> 458.5 mm, vias 0 -> 4
- net areg_out14: track 90.0 -> 261.9 mm
- net alu_neg: track 0.00 -> 171.1 mm, vias 0 -> 5
- net areg_out11: track 85.4 -> 255.3 mm
- net inst_5: track 286.6 -> 451.2 mm, vias 0 -> 4
- net areg_out13: track 102.7 -> 263.0 mm
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- added copper zone on B.Cu, net +3V3
- added copper zone on F.Cu, net GND
Other:
- board outline added: 180.3 x 281.9 mm

Commit message: Rom (#3)
* Updated motherboard with ROM OE,WE, and additional address pins

* ROM schematic, layout, routing complete.
Connections:
- J10 pad 1: Net-(J10-Pad1) -> rom_we
- J10 pad 18: GND -> rom_addr15
- J10 pad 19: +3V3 -> GND
- J10 pad 37: GND -> rom_addr16
- J11 pad 2: GND -> rom_oe
- J4 pad 11: Net-(J4-Pad11) -> rom_we
- J4 pad 27: Net-(J4-Pad27) -> rom_addr15
- J4 pad 29: Net-(J4-Pad29) -> rom_oe
- J4 pad 9: GND -> rom_addr16
Routing:
- net rom_oe: track 0.00 -> 338.3 mm, vias 0 -> 1
- net rom_addr16: track 0.00 -> 333.9 mm, vias 0 -> 1
- net rom_addr15: track 0.00 -> 327.2 mm, vias 0 -> 1
- net rom_we: track 0.00 -> 283.1 mm
- net alu_out15: track 332.9 -> 340.2 mm

Commit message: Ram (#5)
* Flipped clk A and B based on timing diagram. Added output buffers for clock signals.

* Added clock output enable signal to motherboard debugger. Updated component library.

* Schematic and layout for RAM board complete.

* ALU schematic complete, ready for layout and routing.

* ALU layout, routing complete. Associated motherboard mod. 

* Added Load LED to register and program counter boards.
Connections:
- J11 pad 1: +3V3 -> GND
- J11 pad 20: GND -> clk_oe
- J6 pad 5: Net-(J6-Pad5) -> inst_15
- J9 pad 3: Net-(J9-Pad3) -> clk_oe
Routing:
- net clk_oe: track 0.00 -> 297.9 mm, vias 0 -> 1
- net inst_15: track 684.6 -> 762.4 mm, vias 20 -> 21

Commit message: Readme updates (#6)
* Readme intro section

* Board revisions for manufacturing, add digikey PNs to all, added logo.
Parts:
- added G***: LOGO, nandirl logo:logo, F.Cu at (400.7, 165.7)
- J1, J10, J11, J2, J3, J4, J5, J7: footprint Connector_Dsub:DSUB-37_Female_Horizontal_P2.77x2.84mm_EdgePinOffset4.94mm_Housed_MountingHolesOffset7.48mm -> Connector_Dsub:DSUB-37_Female_Horizontal_P2.77x2.84mm_EdgePinOffset7.70mm_Housed_MountingHolesOffset9.12mm
- J6, J8: footprint Connector_Dsub:DSUB-25_Female_Horizontal_P2.77x2.84mm_EdgePinOffset4.94mm_Housed_MountingHolesOffset7.48mm -> Connector_Dsub:DSUB-25_Female_Horizontal_P2.77x2.84mm_EdgePinOffset7.70mm_Housed_MountingHolesOffset9.12mm
- J9: footprint Connector_Dsub:DSUB-9_Female_Horizontal_P2.77x2.84mm_EdgePinOffset4.94mm_Housed_MountingHolesOffset7.48mm -> Connector_Dsub:DSUB-9_Female_Horizontal_P2.77x2.84mm_EdgePinOffset7.70mm_Housed_MountingHolesOffset9.12mm
Other:
- board text added: "Motherboard"
- board text added: "v1.0"

Commit message: Added debugger, schematic and pcb complete.
Routing:
- net (no net): vias 0 -> 6
Changed lines of the file:
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@@
     (thickness 1.6)
     (drawings 6)
-    (tracks 2848)
+    (tracks 2854)
     (zones 0)
     (modules 54)
@@
   (page A2)
   (layers
-    (0 F.Cu signal hide)
+    (0 F.Cu signal)
     (1 In1.Cu signal)
     (2 In2.Cu signal)
-    (31 B.Cu signal hide)
+    (31 B.Cu signal)
     (32 B.Adhes user)
     (33 F.Adhes user)
@@
     (via_min_size 0.4)
     (via_min_drill 0.3)
+    (user_via 6 3.2)
     (uvia_size 0.3)
     (uvia_drill 0.1)
@@
   (gr_line (start 487.68 35.56) (end 487.68 317.5) (layer Edge.Cuts) (width 0.05))
   (gr_line (start 307.34 35.56) (end 487.68 35.56) (layer Edge.Cuts) (width 0.05))
+  (via (at 482.6 40.64) (size 6) (drill 3.2) (layers F.Cu B.Cu) (net 0))
+  (via (at 312.42 40.64) (size 6) (drill 3.2) (layers F.Cu B.Cu) (net 0))
+  (via (at 482.6 312.42) (size 6) (drill 3.2) (layers F.Cu B.Cu) (net 0))
+  (via (at 322.58 312.42) (size 6) (drill 3.2) (layers F.Cu B.Cu) (net 0))
+  (via (at 394.97 114.3) (size 6) (drill 3.2) (layers F.Cu B.Cu) (net 0))
+  (via (at 394.97 218.44) (size 6) (drill 3.2) (layers F.Cu B.Cu) (net 0))
   (segment (start 338.17 311.335) (end 338.17 309.88) (width 0.25) (layer F.Cu) (net 1))
   (segment (start 339.555 312.72) (end 338.17 311.335) (width 0.25) (layer F.Cu) (net 1))
