File: kicad/ram/Dlatch_16bit.sch (KiCad schematic (older format))
At the start: 16 parts, among them U39 SN74ALVC00, U40 SN74ALVC00, U41 SN74ALVC00, U42 SN74ALVC00, U43 SN74ALVC00, U44 SN74ALVC00, U45 SN74ALVC00, U46 SN74ALVC00, U47 SN74ALVC00, U48 SN74ALVC00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

Commit message: Readme updates (#6)
* Readme intro section

* Board revisions for manufacturing, add digikey PNs to all, added logo.
Parts:
- U39, U40, U41, U42, U43, U44, U45, U46, U47, U48, U49, U50, U51, U52, U53, U54: Digikey PN (none) -> 296-5104-1-ND
