File: kicad/ram/ram.kicad_pcb (KiCad board)
At the start: 4 copper layers, 102.9 x 133.3 mm, 64 parts, among them J1 I/O Expansion 1, J2 I/O Expansion 2, J3 DB25_Male, J4 DB37_Male, U1 71V016SA12PHGI, U10 SN74ALVC00, U11 SN74ALVC00, U12 SN74ALVC00, U13 SN74ALVC00, U14 SN74ALVC00, U15 SN74ALVC00, U16 SN74ALVC00, U17 SN74ALVC00, U18 SN74ALVC00, U19 SN74ALVC00, U2 SN74ALVC00, U20 SN74ALVC00, U21 SN74ALVC00, U22 SN74ALVC00, U23 SN74ALVC00, U24 SN74ALVC00, U25 SN74ALVC00, U26 SN74ALVC00, U27 SN74ALVC00, U28 SN74ALVC00, U29 SN74ALVC00, U3 SN74ALVC00, U30 SN74ALVC00, U31 SN74ALVC00, U32 SN74ALVC00, U33 SN74ALVC00, U34 SN74ALVC00, U35 SN74ALVC00, U36 SN74ALVC00, U37 SN74ALVC00, U38 SN74ALVC00, U39 SN74ALVC00, U4 SN74ALVC00, U40 SN74ALVC00, U41 SN74ALVC00, U42 SN74ALVC00, U43 SN74ALVC00, U44 SN74ALVC00, U45 SN74ALVC00, U46 SN74ALVC00, U47 SN74ALVC00, U48 SN74ALVC00, U49 SN74ALVC00, U5 SN74LVC541APWR, U50 SN74ALVC00, U51 SN74ALVC00, U52 SN74ALVC00, U53 SN74ALVC00, U54 SN74ALVC00, U6 SN74LVC541APWR, U7 SN74ALVC00, U8 SN74ALVC00, U9 SN74ALVC00

Commit message: Readme updates (#6)
* Readme intro section

* Board revisions for manufacturing, add digikey PNs to all, added logo.
Parts:
- added G***: LOGO, nandirl logo:logo_sm, F.Cu at (225.4, 15.9)
- J3: footprint Connector_Dsub:DSUB-25_Male_Horizontal_P2.77x2.84mm_EdgePinOffset4.94mm_Housed_MountingHolesOffset7.48mm -> Connector_Dsub:DSUB-25_Male_Horizontal_P2.77x2.84mm_EdgePinOffset7.70mm_Housed_MountingHolesOffset9.12mm
- J4: footprint Connector_Dsub:DSUB-37_Male_Horizontal_P2.77x2.84mm_EdgePinOffset4.94mm_Housed_MountingHolesOffset7.48mm -> Connector_Dsub:DSUB-37_Male_Horizontal_P2.77x2.84mm_EdgePinOffset7.70mm_Housed_MountingHolesOffset9.12mm
Other:
- board text added: "RAM"
- board text added: "v1.0"
- board text removed: "Memory-Mapped I/O"
- board text removed: "Random Access Memory"
