File: kicad/ram/ram.sch (KiCad schematic (older format))
At the start: 16 parts, among them J1 I/O Expansion 1, J2 I/O Expansion 2, J3 DB25_Male, J4 DB37_Male, U1 71V016SA12PHGI, U2 SN74ALVC00, U3 SN74ALVC00, U4 SN74ALVC00, U5 SN74LVC541APWR, U6 SN74LVC541APWR

Commit message: Readme updates (#6)
* Readme intro section

* Board revisions for manufacturing, add digikey PNs to all, added logo.
Parts:
- C5, C6: Digikey PN (none) -> 399-C1206C104K5RAC7800CT-ND
- J3: footprint Connector_Dsub:DSUB-25_Male_Horizontal_P2.77x2.84mm_EdgePinOffset4.94mm_Housed_MountingHolesOffset7.48mm -> Connector_Dsub:DSUB-25_Male_Horizontal_P2.77x2.84mm_EdgePinOffset7.70mm_Housed_MountingHolesOffset9.12mm; Digikey PN (none) -> AE10980-ND
- J4: footprint Connector_Dsub:DSUB-37_Male_Horizontal_P2.77x2.84mm_EdgePinOffset4.94mm_Housed_MountingHolesOffset7.48mm -> Connector_Dsub:DSUB-37_Male_Horizontal_P2.77x2.84mm_EdgePinOffset7.70mm_Housed_MountingHolesOffset9.12mm; Digikey PN (none) -> AE10986-ND
Changed lines of the file:
@@
 F 0 "J4" H 10818 658 50  0000 C CNN
 F 1 "DB37_Male" H 10818 749 50  0000 C CNN
-F 2 "Connector_Dsub:DSUB-37_Male_Horizontal_P2.77x2.84mm_EdgePinOffset4.94mm_Housed_MountingHolesOffset7.48mm" H 10900 2750 50  0001 C CNN
+F 2 "Connector_Dsub:DSUB-37_Male_Horizontal_P2.77x2.84mm_EdgePinOffset7.70mm_Housed_MountingHolesOffset9.12mm" H 10900 2750 50  0001 C CNN
 F 3 " ~" H 10900 2750 50  0001 C CNN
+F 4 "AE10986-ND" H 10900 2750 50  0001 C CNN "Digikey PN"
 	1    10900 2750
 	1    0    0    -1
@@
 F 0 "J3" H 9850 3700 50  0000 L CNN
 F 1 "DB25_Male" H 9800 3600 50  0000 L CNN
-F 2 "Connector_Dsub:DSUB-25_Male_Horizontal_P2.77x2.84mm_EdgePinOffset4.94mm_Housed_MountingHolesOffset7.48mm" H 9900 2150 50  0001 C CNN
+F 2 "Connector_Dsub:DSUB-25_Male_Horizontal_P2.77x2.84mm_EdgePinOffset7.70mm_Housed_MountingHolesOffset9.12mm" H 9900 2150 50  0001 C CNN
 F 3 " ~" H 9900 2150 50  0001 C CNN
+F 4 "AE10980-ND" H 9900 2150 50  0001 C CNN "Digikey PN"
 	1    9900 2150
 	1    0    0    -1
@@
 F 2 "Capacitor_SMD:C_1206_3216Metric" H 2950 1850 50  0001 C CNN
 F 3 "~" H 2950 1850 50  0001 C CNN
+F 4 "399-C1206C104K5RAC7800CT-ND" V 2950 1850 50  0001 C CNN "Digikey PN"
 	1    2950 1850
 	0    1    1    0
@@
 F 2 "Capacitor_SMD:C_1206_3216Metric" H 850 1850 50  0001 C CNN
 F 3 "~" H 850 1850 50  0001 C CNN
+F 4 "399-C1206C104K5RAC7800CT-ND" H 850 1850 50  0001 C CNN "Digikey PN"
 	1    850  1850
 	-1   0    0    1
