File: kicad/rom/rom.kicad_pcb (KiCad board)
At the start: 2 copper layers, 72.4 x 47 mm, 8 parts, among them J1 DB37_Male, U1 SST39VF200A

Commit message: Readme updates (#6)
* Readme intro section

* Board revisions for manufacturing, add digikey PNs to all, added logo.
Parts:
- added G***: LOGO, nandirl logo:logo_sm, F.Cu at (145.0, 80.8)
- J1: footprint Connector_Dsub:DSUB-37_Male_Horizontal_P2.77x2.84mm_EdgePinOffset4.94mm_Housed_MountingHolesOffset7.48mm -> Connector_Dsub:DSUB-37_Male_Horizontal_P2.77x2.84mm_EdgePinOffset7.70mm_Housed_MountingHolesOffset9.12mm
Other:
- board text added: "ROM"
- board text added: "v1.0"
- board text removed: "Read-Only Memory"
