File: hardware/program_counter/program_counter.kicad_pcb (KiCad board)
At the start: 4 copper layers, 175.3 x 72.4 mm, 111 parts, among them J1 DB37_Male, U1 SN74HCS00PWR, U10 SN74HCS00PWR, U11 SN74HCS00PWR, U12 SN74HCS00PWR, U13 SN74HCS00PWR, U14 SN74HCS00PWR, U15 SN74HCS00PWR, U16 SN74HCS00PWR, U17 SN74HCS00PWR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

Commit message: All boards as fabbed at v1.0
Parts:
- added G***: LOGO, nandirl logo:logo_sm, F.Cu at (234.9, 83.8)
